File: 9bay_sata_backplane.kicad_sch (KiCad schematic)
At the start: 57 parts, among them J1 Screw_Terminal_01x04, U1 SATA_Connector, U10 SATA_Data, U11 SATA_Data, U12 SATA_Data, U13 SATA_Data, U14 SATA_Data, U15 SATA_Data, U16 SATA_Data, U17 SATA_Data, U18 SATA_Data, U2 SATA_Connector, U3 SATA_Connector, U4 SATA_Connector, U5 SATA_Connector, U6 SATA_Connector, U7 SATA_Connector, U8 SATA_Connector, U9 SATA_Connector

Commit message: DIY 9-Bay SATA Backplane v1.2
Parts:
- removed C10, C11, C12, C13, C14, C15, C16, C17, C18, C2, C3, C4, C5, C6, C7, C8, C9: C_Small, Capacitor_SMD:C_1206_3216Metric, symbol Device:C_Small
- removed C19, C20: C_Polarized_Small, Capacitor_THT:C_Radial_D16.0mm_H25.0mm_P7.50mm, symbol Device:C_Polarized_Small
- removed J1: Screw_Terminal_01x04, TerminalBlock:TerminalBlock_Xinya_XY308-2.54-4P_1x04_P2.54mm_Horizontal, symbol Connector:Screw_Terminal_01x04
- removed R1, R10, R11, R12, R13, R14, R15, R16, R17, R18, R2, R3, R4, R5, R6, R7, R8, R9: R_Small_US, Resistor_SMD:R_1206_3216Metric, symbol Device:R_Small_US
- removed U1, U2, U3, U4, U5, U6, U7, U8, U9: SATA_Connector, Connector_SATA_SAS:CONN_877791001_MOL, symbol sata_connector:sata_22pin
- removed U10, U11, U12, U13, U14, U15, U16, U17, U18: SATA_Data, Connector_SATA_SAS:CONN_67800-8025_MOL, symbol sata_connector:sata_7pin
- added C1, C2: 25v 560uf, Capacitor_THT:CP_Radial_D10.0mm_P5.00mm, symbol Device:C_Polarized
- added C201, C301, C401, C501, C601, C701, C801, C901: 35v 10uf, Capacitor_SMD:C_1206_3216Metric, symbol Device:C_Small
- added H1, H2, H3, H4, H5, H6: MountingHole, MountingHole:MountingHole_3mm, symbol Mechanical:MountingHole
- added J1: HDD POWER, Connector_TE-Connectivity:TE_MATE-N-LOK_350211-1_1x04_P5.08mm_Vertical, symbol Connector_Generic:Conn_01x04
- added J101, J201, J301, J401, J501, J601, J701, J801, J901: 87779-1001, 87779-1001:877791001, symbol 87779-1001:87779-1001_1
- added J102, J202, J302, J402, J502, J602, J702, J802, J902: 67800-8025, 67800-8025:678008025, symbol 67800-8025:67800-8025
- added R101, R201, R301, R401, R501, R601, R701, R801, R901: 22ohm, Resistor_SMD:R_1206_3216Metric, symbol Device:R
- C101: renamed from C1; value C_Small -> 35v 10uf
Connections:
- net +5V: now also C1.1, C2.1, C201.2, C301.2, C401.2, C501.2, C601.2, C701.2, C801.2, C901.2, J1.4 (Pin_4), J101.P8, J101.P9, J201.P8, J201.P9, J301.P8, J301.P9, J401.P8, J401.P9, J501.P8, J501.P9, J601.P8, J601.P9, J701.P8, J701.P9, J801.P8, J801.P9, J901.P8, J901.P9, R101.2, R201.2, R301.2, R401.2, R501.2, R601.2, R701.2, R801.2, R901.2
- net GND: now also C1.2, C2.2, C201.1, C301.1, C401.1, C501.1, C601.1, C701.1, C801.1, C901.1, J1.2 (Pin_2), J1.3 (Pin_3), J101.P10, J101.P11, J101.P12, J101.P4, J101.P5, J101.P6, J101.S1, J101.S4, J101.S7, J102.1, J102.4, J102.7, J201.P10, J201.P11, J201.P12, J201.P4, J201.P5, J201.P6, J201.S1, J201.S4, J201.S7, J202.1, J202.4, J202.7, J301.P10, J301.P11, J301.P12, J301.P4, J301.P5, J301.P6, J301.S1, J301.S4, J301.S7, J302.1, J302.4, J302.7, J401.P10, J401.P11, J401.P12, J401.P4, J401.P5, J401.P6, J401.S1, J401.S4, J401.S7, J402.1, J402.4, J402.7, J501.P10, J501.P11, J501.P12, J501.P4, J501.P5, J501.P6, J501.S1, J501.S4, J501.S7, J502.1, J502.4, J502.7, J601.P10, J601.P11, J601.P12, J601.P4, J601.P5, J601.P6, J601.S1, J601.S4, J601.S7, J602.1, J602.4, J602.7, J701.P10, J701.P11, J701.P12, J701.P4, J701.P5, J701.P6, J701.S1, J701.S4, J701.S7, J702.1, J702.4, J702.7, J801.P10, J801.P11, J801.P12, J801.P4, J801.P5, J801.P6, J801.S1, J801.S4, J801.S7, J802.1, J802.4, J802.7, J901.P10, J901.P11, J901.P12, J901.P4, J901.P5, J901.P6, J901.S1, J901.S4, J901.S7, J902.1, J902.4, J902.7
- new net: J901.P7, R901.1
- new net: J601.P7, R601.1
- new net: J501.P7, R501.1
- new net: J401.P7, R401.1
- new net: J801.P7, R801.1
- new net: J301.P7, R301.1
- new net: J701.P7, R701.1
- new net: J201.P7, R201.1
- new net: J101.P7, R101.1
- new net SATA1 A+: J101.S2, J102.2
- new net SATA1 A-: J101.S3, J102.3
- new net SATA1 B+: J101.S6, J102.6
- new net SATA1 B-: J101.S5, J102.5
- new net SATA2 A+: J201.S2, J202.2
- new net SATA2 A-: J201.S3, J202.3
- new net SATA2 B+: J201.S6, J202.6
- new net SATA2 B-: J201.S5, J202.5
- new net SATA3 A+: J301.S2, J302.2
- new net SATA3 A-: J301.S3, J302.3
- new net SATA3 B+: J301.S6, J302.6
- new net SATA3 B-: J301.S5, J302.5
- new net SATA4 A+: J401.S2, J402.2
- new net SATA4 A-: J401.S3, J402.3
- new net SATA4 B+: J401.S6, J402.6
- new net SATA4 B-: J401.S5, J402.5
- new net SATA5 A+: J501.S2, J502.2
- new net SATA5 A-: J501.S3, J502.3
- new net SATA5 B+: J501.S6, J502.6
- new net SATA5 B-: J501.S5, J502.5
- new net SATA6 A+: J601.S2, J602.2
- new net SATA6 A-: J601.S3, J602.3
- new net SATA6 B+: J601.S6, J602.6
- new net SATA6 B-: J601.S5, J602.5
- new net SATA7 A+: J701.S2, J702.2
- new net SATA7 A-: J701.S3, J702.3
- new net SATA7 B+: J701.S6, J702.6
- new net SATA7 B-: J701.S5, J702.5
- new net SATA8 A+: J801.S2, J802.2
- new net SATA8 A-: J801.S3, J802.3
- new net SATA8 B+: J801.S6, J802.6
- new net SATA8 B-: J801.S5, J802.5
- new net SATA9 A+: J901.S2, J902.2
- new net SATA9 A-: J901.S3, J902.3
- new net SATA9 B+: J901.S6, J902.6
- new net SATA9 B-: J901.S5, J902.5
- no-connect marks 0 -> 75
Other:
- note added: "SATA Port 1"
- note added: "SATA Port 2"
- note added: "SATA Port 3"
- note added: "SATA Port 4"
- note added: "SATA Port 5"
- note added: "SATA Port 6"
- note added: "SATA Port 7"
- note added: "SATA Port 8"
- note added: "SATA Port 9"
- company: (none) -> FreudianNonce
- title: (none) -> DIY 9 Bay SATA Backplane
- moved on the sheet: C101
